File: PCB Design/Power_Motor_Board/Power_Motor_Board.kicad_sch (KiCad schematic)
At the start: 25 parts, among them IC2 AP63205WU-7, IC3 DRV8251ADDAR, J1 691137710002, J2A1 SSW-119-01-T-D, J2B1 SSW-119-01-T-D

Commit message: Majority of schematic built
Bluetooth module part left to build
Parts:
- removed D4: LED_Filled, LED_SMD:LED_0603_1608Metric_Pad1.05x0.95mm_HandSolder, symbol Device:LED_Filled
- removed J2B1: SSW-119-01-T-D, symbol SamacSys_Parts:SSW-119-01-T-D_1
- removed Motor_Connecter: 691137710002, Connector_PinSocket_2.54mm:PinSocket_1x02_P2.54mm_Vertical, symbol SamacSys_Parts:691137710002
- removed R4: 1.1kΩ, Resistor_SMD:R_0603_1608Metric_Pad0.98x0.95mm_HandSolder, symbol Device:R_US
- removed TP1: TestPoint, symbol Connector:TestPoint
- added C13: 10nF, Capacitor_SMD:C_1206_3216Metric_Pad1.33x1.80mm_HandSolder, symbol Device:C
- added C14, C15, C18: 0.1uF, Capacitor_SMD:C_1206_3216Metric_Pad1.33x1.80mm_HandSolder, symbol Device:C
- added C16: 180uF, Capacitor_SMD:C_1206_3216Metric_Pad1.33x1.80mm_HandSolder, symbol Device:C_Polarized
- added C17: 10uF, Capacitor_SMD:C_1206_3216Metric_Pad1.33x1.80mm_HandSolder, symbol Device:C
- added C19, C20: 22uF, Capacitor_SMD:C_1210_3225Metric_Pad1.33x2.70mm_HandSolder, symbol Device:C
- added IC1: DRV8251ADDAR, RC Car Motor Driver Board Workshop:SOIC-8-DDA-DRV8231_TEX, symbol SamacSys_Parts:DRV8251ADDAR
- added IC4: AP63205WU-7, Package_TO_SOT_SMD:TSOT-23-6_HandSoldering, symbol SamacSys_Parts:AP63205WU-7
- added J2, J3: 691137710002, FootPrintLibrary_ENEL300:SHDR2W70P0X500_1X2_1000X750X1150P, symbol SamacSys_Parts:691137710002
- added J4: Conn_01x06, Connector_PinSocket_2.54mm:PinSocket_1x06_P2.54mm_Horizontal, symbol Connector_Generic:Conn_01x06
- added L2: 4.7uH, Inductor_SMD:L_Wuerth_XHMI-6060, symbol SamacSys_Parts:IFSC2020DEER4R7M01
- added R1: 0Ω, Resistor_SMD:R_1206_3216Metric_Pad1.30x1.75mm_HandSolder, symbol Device:R_US
- added R2: 750Ω, Resistor_SMD:R_1206_3216Metric_Pad1.30x1.75mm_HandSolder, symbol Device:R_US
- added TP1, TP2: 5019, FootPrintLibrary_ENEL300:5019, symbol SamacSys_Parts:5019
- C10, C11, C12, C2, C5, C6, C7, C8, C9: footprint Capacitor_SMD:C_0603_1608Metric_Pad1.08x0.95mm_HandSolder -> Capacitor_SMD:C_1206_3216Metric_Pad1.33x1.80mm_HandSolder
- F1: value 5A -> 4A
- J1: footprint (none) -> FootPrintLibrary_ENEL300:SHDR2W70P0X500_1X2_1000X750X1150P
- J2A1: footprint RC Car Motor Driver Board Workshop:STM_Nucleo_Morpho_x2_Footprint -> FootPrintLibrary_ENEL300:STM_Nucleo_Morpho_x2_Footprint
- L1: value IFSC2020DEER4R7M01 -> 4.7uH
- R3, R7: footprint Resistor_SMD:R_0603_1608Metric_Pad0.98x0.95mm_HandSolder -> Resistor_SMD:R_1206_3216Metric_Pad1.30x1.75mm_HandSolder
Connections:
- net +3V3: now also C14.1, IC1.4 (VREF)
- net +5V: now also C19.2, C20.2, IC4.1 (FB), L2.2, TP1.1, TP2.1; no longer C1.2, C10.2, C11.2, C12.2, C3.1, C4.1, C5.2, C6.2, C7.2, C8.2, C9.2, IC2.4 (GND), IC3.7 (GND_1), IC3.9 (GND_2), J1.2, J2A1.A10 (NC), J2A1.A12 (IOREF), J2A1.A19 (GND), J2A1.A20 (GND), J2A1.A22 (GND), J2A1.A8 (GND), R7.2
- net +OUT: now also IC1.6 (OUT1), J2.2, J3.2
- net +Vbatt: now also C17.1, IC4.2 (EN), IC4.3 (VIN)
- net -OUT: now also IC1.8 (OUT2), J2.1, J3.1
- net IN1_MTR1: now also J2A1.B21 (PA9), IC1.3 (IN1); no longer IC3.3 (IN1), J2A1.A38 (PC0)
- net IN2-MTR1: now also J2A1.B23 (PA8), IC1.2 (IN2); no longer IC3.2 (IN2), J2A1.A36 (PC1)
- net Vbatt: now reaches C6.1, C8.1, IC3.5 (VM)
- net Vbatt: now also C15.1, C16.1, IC1.5 (VM)
- net at J2A1.A35 (PC2): now also R1.1; no longer R3.1
- net I_MTR2: now reaches J2A1.A37 (PC3)
- net I_MTR2: now also R3.1
- new net: C18.1, IC4.5 (SW), L2.1
- new net: C13.1, IC1.1 (IPROPI), R1.2, R2.1
- new net: C18.2, IC4.6 (BST)
- new net: J2A1., J2A1.B36 (NC)
- new net BT_RX: J4.3 (Pin_3)
- new net BT_TX: J4.2 (Pin_2)
- new net GND: C1.2, C10.2, C11.2, C12.2, C13.2, C14.2, C15.2, C16.2, C17.2, C19.1, C20.1, C3.1, C4.1, C5.2, C6.2, C7.2, C8.2, C9.2, IC1.7 (GND_1), IC1.9 (GND_2), IC2.4 (GND), IC3.7 (GND_1), IC3.9 (GND_2), IC4.4 (GND), J1.2, J2A1.A19 (GND), J2A1.A20 (GND), J2A1.A22 (GND), J2A1.A8 (GND), J2A1.B20 (GND), J2A1.B9 (GND), J4.6 (Pin_6), R2.2, R7.2
- new net IN1_MTR2: IC3.3 (IN1), J2A1.B33 (PA10)
- new net IN2_MTR2: IC3.2 (IN2), J2A1.B14 (PA11)
- new net VDD: J4.1 (Pin_1)
Other:
- note added: "5V Regulated Supply (Drivers)"
- note added: "5V Regulated Supply (Nucleo Board)"
- note added: "Left"
- note added: "Motor Drivers"
- note added: "NOTE WHERE +ve and -ve is!!!!"
- note added: "Nucleo Board"
- note added: "Right"
- note removed: "5V Regulated Supply"
- moved on the sheet: C1, C10, C11, C12, C2, C3, C5, C6, C7, C8, C9, F1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

Commit message: Completed Schematic
Parts:
- IC1, IC3: footprint RC Car Motor Driver Board Workshop:SOIC-8-DDA-DRV8231_TEX -> FootPrintLibrary_ENEL300:SOIC-8-DDA-DRV8231_TEX
Connections:
- net +5V: now also J4.5 (Pin_5)
- net BT_RX: now also J2A1.A28 (PA0), J4.2 (Pin_2); no longer J4.3 (Pin_3)
- net BT_TX: now also J2A1.A30 (PA1), J4.3 (Pin_3); no longer J4.2 (Pin_2)
- net GND: now also J4.4 (Pin_4); no longer J4.6 (Pin_6)
- net VDD renamed State
- new net EN: J4.6 (Pin_6)
Other:
- note added: "Bluetooth Module"
- moved on the sheet: J4

Commit message: Rough draft of the layout is completed
Connections:
- net I_MTR1: now reaches J2A1.A35 (PC2), R1.1

Commit message: Updates
Parts:
- J4: footprint Connector_PinSocket_2.54mm:PinSocket_1x06_P2.54mm_Horizontal -> Connector_PinSocket_2.54mm:PinSocket_1x06_P2.54mm_Vertical
Changed lines of the file:
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@@
 			)
 		)
-		(property "Footprint" "Connector_PinSocket_2.54mm:PinSocket_1x06_P2.54mm_Horizontal"
+		(property "Footprint" "Connector_PinSocket_2.54mm:PinSocket_1x06_P2.54mm_Vertical"
 			(at 264.16 190.5 0)
 			(effects

Commit message: First Revision of Power_Motor PCB
Parts:
- added H1, H2, H3, H4: MountingHole, MountingHole:MountingHole_3.2mm_M3, symbol Mechanical:MountingHole
Connections:
- net +5V: no longer C3.2, C4.2, IC2.1 (FB), L1.2, TP1.1
- net +OUT renamed +OUT_1
- net +OUT_1: no longer IC3.6 (OUT1), J2.2
- net -OUT renamed -OUT_1
- net -OUT_1: no longer IC3.8 (OUT2), J2.1
- net Vbatt renamed 5V
- net 5V: now also C3.2, C4.2, IC2.1 (FB), L1.2, TP1.1
- new net +OUT_2: IC3.6 (OUT1), J2.2
- new net -OUT_2: IC3.8 (OUT2), J2.1
Other:
- moved on the sheet: J4

Commit message: Started assigning Manufacture Part Numbers
Parts:
- C1, C17: Manufacture Part Number (none) -> CL31B106KAHNNNE
- C10, C12: Manufacture Part Number (none) -> CL31B105KBHNNNE
- C11, C14, C15, C18, C2, C7, C8, C9: Manufacture Part Number (none) -> C1206C104K5RACTU
- C13, C5: Manufacture Part Number (none) -> C1206C103K5RACTU
- C19, C20, C3, C4: Manufacture Part Number (none) -> CL32A226KAJNNNE
- F1: Manufacture Part Number (none) -> 0685T4000-01
- IC1, IC3: Manufacture Part Number (none) -> DRV8251ADDAR
- IC2, IC4: Manufacture Part Number (none) -> AP63205WU-7
- L1, L2: Manufacture Part Number (none) -> IFSC2020DEER4R7M01

Commit message: Finished assigning part numbers
Parts:
- C16, C6: Manufacture Part Number (none) -> A768KE187M1ELAE029
- J1, J2, J3: now left out of the parts list
- R1, R3: Manufacture Part Number (none) -> RC1206JR-070RL
- R2, R7: Manufacture Part Number (none) -> RC1206FR-07750RL
- TP1, TP2: now not fitted; now left out of the parts list
Changed lines of the file:
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@@
 			)
 		)
-		(property "Manufacture Part Number" ""
+		(property "Manufacture Part Number" "RC1206FR-07750RL"
 			(at 124.46 137.16 0)
 			(effects
@@
 		(unit 1)
 		(exclude_from_sim no)
-		(in_bom yes)
+		(in_bom no)
 		(on_board yes)
-		(dnp no)
+		(dnp yes)
 		(fields_autoplaced yes)
 		(property "Reference" "TP1"
@@
 			)
 		)
-		(property "Manufacture Part Number" ""
+		(property "Manufacture Part Number" "A768KE187M1ELAE029"
 			(at 205.74 68.58 0)
 			(effects
@@
 		(unit 1)
 		(exclude_from_sim no)
-		(in_bom yes)
+		(in_bom no)
 		(on_board yes)
 		(dnp no)
@@
 		(unit 1)
 		(exclude_from_sim no)
-		(in_bom yes)
+		(in_bom no)
 		(on_board yes)
 		(dnp no)
@@
 			)
 		)
-		(property "Manufacture Part Number" ""
+		(property "Manufacture Part Number" "RC1206JR-070RL"
 			(at 120.65 48.26 90)
 			(effects
@@
 		(unit 1)
 		(exclude_from_sim no)
-		(in_bom yes)
+		(in_bom no)
 		(on_board yes)
-		(dnp no)
+		(dnp yes)
 		(fields_autoplaced yes)
 		(property "Reference" "TP2"
@@
 			)
 		)
-		(property "Manufacture Part Number" ""
+		(property "Manufacture Part Number" "RC1206JR-070RL"
 			(at 114.3 115.57 90)
 			(effects
@@
 		(unit 1)
 		(exclude_from_sim no)
-		(in_bom yes)
+		(in_bom no)
 		(on_board yes)
 		(dnp no)
@@
 			)
 		)
-		(property "Manufacture Part Number" ""
+		(property "Manufacture Part Number" "RC1206FR-07750RL"
 			(at 130.81 69.85 0)
 			(effects
@@
 			)
 		)
-		(property "Manufacture Part Number" ""
+		(property "Manufacture Part Number" "A768KE187M1ELAE029"
 			(at 199.39 135.89 0)
 			(effects

Commit message: Finished BOM list and updated layout to use the correct 180uF capacitor footprint
Parts:
- C16, C6: footprint Capacitor_SMD:C_1206_3216Metric_Pad1.33x1.80mm_HandSolder -> FootPrintLibrary_ENEL300:A768KE187M1ELAE029
Changed lines of the file:
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@@
 			)
 		)
-		(property "Footprint" "Capacitor_SMD:C_1206_3216Metric_Pad1.33x1.80mm_HandSolder"
+		(property "Footprint" "FootPrintLibrary_ENEL300:A768KE187M1ELAE029"
 			(at 206.7052 72.39 0)
 			(effects
@@
 			)
 		)
-		(property "Footprint" "Capacitor_SMD:C_1206_3216Metric_Pad1.33x1.80mm_HandSolder"
+		(property "Footprint" "FootPrintLibrary_ENEL300:A768KE187M1ELAE029"
 			(at 200.3552 139.7 0)
 			(effects
