File: PCB Design/Power_Motor_Board_v2/Power_Motor_Board_v2.kicad_sch (KiCad schematic)
At the start: 38 parts, among them IC1 DRV8251ADDAR, IC3 DRV8251ADDAR, IC4 AP63205WU-7, J1 691137710002, J2 691137710002, J2A1 SSW-119-01-T-D, J3 691137710002, J4 Conn_01x06, J5 Conn_01x02_Socket

Commit message: personal notes for future, and changes to the schmatic
i forgot my changes icl. idk if i mentioned adding the metal detector connector pins that connect to 5V and GND
Parts:
- J5: footprint (none) -> Connector_PinSocket_2.54mm:PinSocket_1x02_P2.54mm_Vertical
- R4, R5: footprint (none) -> Resistor_SMD:R_1206_3216Metric_Pad1.30x1.75mm_HandSolder
Connections:
- net GND: now also J5.2 (Pin_2)
- net VDD: now reaches J5.1 (Pin_1)
Other:
- note added: "- coordinate MD 5v gnd to main board 5v and gnd"
- note added: "- order x2 components - order MD components - double check schematics and parts"
- moved on the sheet: F1, J1, J4, J5, R4, R5
