File: PCB Design/Metal_Detector/Metal_Detector.kicad_sch (KiCad schematic)
At the start: 0 parts

Commit message: made the metal detector schematic with the amazingamy
Parts:
- added BZ1: Buzzer, symbol Device:Buzzer
- added C1: 100nF, symbol Device:C
- added C2: C, symbol Device:C
- added J1, J2: Conn_01x01_Socket, symbol Connector:Conn_01x01_Socket
- added Q1: 2N3904, symbol Transistor_BJT:BC107
- added R1, R3: 1kΩ, symbol Device:R
- added R2: 33kΩ, symbol Device:R
- added U1: 555 Timer, Package_SO:SOIC-8_3.9x4.9mm_P1.27mm, symbol Timer:ICM7555xB
Connections:
- new net: R2.2, R3.1, U1.7 (DISCH)
- new net: C2.2, U1.5 (CONT)
- new net: Q1.2 (B), R1.1
- new net: C1.1, R2.1, U1.2 (TRIG), U1.6 (THRES)
- new net: BZ1.1 (+), Q1.3 (C)
- new net: BZ1.2 (-), J1.1 (Pin_1)
- new net Buzzer: R1.2, U1.3 (OUT)
- new net GND: C1.2, C2.1, Q1.1 (E), U1.1 (GND)
- new net VDD: J2.1 (Pin_1), R3.2, U1.4 (~{RST}), U1.8 (VCC)
Other:
- note added: "2/27/26"
- note added: "555 Timer"
- note added: "Buzzer"
- note added: "Metal Detector"

Commit message: added connector for voltage? thingy (5V + GND)
Parts:
- added J3: Conn_01x02_Pin, symbol Connector:Conn_01x02_Pin
- C2: value C -> 1μF
Connections:
- net GND: now also J3.2 (Pin_2)
- net VDD renamed +5V
- net +5V: now also J3.1 (Pin_1)
Other:
- note added: "Connector"
- moved on the sheet: BZ1, C1, C2, J1, J2, Q1, R1, R2, R3, U1

Commit message: did all the footprints w amy chan
Parts:
- removed J1, J2: Conn_01x01_Socket, symbol Connector:Conn_01x01_Socket
- added J2: Conn_01x02_Socket, Connector_PinSocket_2.54mm:PinSocket_1x02_P2.54mm_Vertical, symbol Connector:Conn_01x02_Socket
- BZ1: footprint (none) -> Buzzer_Beeper:Buzzer_12x9.5RM7.6; now left out of the parts list
- C1: footprint (none) -> Capacitor_SMD:C_0805_2012Metric_Pad1.18x1.45mm_HandSolder; Manufacture Product Number (none) -> C0805F104K1RACAUTO
- C2: value 1μF -> 10nF; footprint (none) -> Capacitor_SMD:C_1206_3216Metric_Pad1.33x1.80mm_HandSolder; Manufacture Product Number (none) -> CHV1206N500103JCT
- J3: footprint (none) -> Connector_PinHeader_2.54mm:PinHeader_1x02_P2.54mm_Vertical; now left out of the parts list
- Q1: footprint (none) -> Package_TO_SOT_THT:TO-92L_Inline; now left out of the parts list
- R1, R3: footprint (none) -> Resistor_SMD:R_1206_3216Metric_Pad1.30x1.75mm_HandSolder; Manufacture Product Number (none) -> RC1206FR-071KL
- R2: footprint (none) -> Resistor_SMD:R_1206_3216Metric_Pad1.30x1.75mm_HandSolder; Manufacture Product Number (none) -> RC1206JR-0733KL
- U1: now left out of the parts list
Connections:
- net +5V: now also J2.1 (Pin_1)
- net Power2: now reaches BZ1.2 (-)
- net Power2: now also J2.2 (Pin_2)
Other:
- note added: "Connection to 5V and GND"
- note added: "Exposed Wires"
- moved on the sheet: C1, C2, J3, R2, R3, U1

Commit message: did layout and traces w amy exported step file
Changed lines of the file:
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@@
-	)
-	(junction
-		(at 165.1 78.74)
-		(diameter 0)
-		(color 0 0 0 0)
 	)
 	(junction
@@
 	(wire
 		(pts
-			(xy 165.1 78.74) (xy 165.1 83.82)
+			(xy 165.1 69.85) (xy 165.1 83.82)
 		)
 		(stroke
@@
 	(wire
 		(pts
-			(xy 165.1 78.74) (xy 171.45 78.74)
-		)
-		(stroke
-			(width 0)
-			(type default)
-		)
-	)
-	(wire
-		(pts
 			(xy 45.72 96.52) (xy 45.72 106.68)
 		)
@@
 		(pts
 			(xy 148.59 83.82) (xy 152.4 83.82)
-		)
-		(stroke
-			(width 0)
-			(type default)
-		)
-	)
-	(wire
-		(pts
-			(xy 165.1 69.85) (xy 165.1 78.74)
 		)
 		(stroke
@@
 	(label "Buzzer"
 		(at 50.8 76.2 0)
-		(effects
-			(font
-				(size 1.27 1.27)
-			)
-			(justify left bottom)
-		)
-	)
-	(label "Power"
-		(at 171.45 78.74 0)
 		(effects
 			(font
@@
 		)
 	)
-	(label "Power"
-		(at 242.57 102.87 0)
-		(effects
-			(font
-				(size 1.27 1.27)
-			)
-			(justify left bottom)
-		)
-	)
 	(symbol
 		(lib_id "Device:R")
@@
 					(unit 1)
 				)
+			)
+		)
+	)
+	(symbol
+		(lib_id "power:VDD")
+		(at 242.57 102.87 0)
+		(unit 1)
+		(exclude_from_sim no)
+		(in_bom yes)
+		(on_board yes)
+		(dnp no)
+		(fields_autoplaced yes)
+		(property "Reference" "#PWR08"
+			(at 242.57 106.68 0)
+			(effects
+				(font
+					(size 1.27 1.27)
+				)
+				(hide yes)
+			)
+		)
+		(property "Value" "+5V"
+			(at 242.57 97.79 0)
+			(effects
+				(font
+					(size 1.27 1.27)
+				)
+			)
+		)
+		(property "Footprint" ""
+			(at 242.57 102.87 0)
+			(effects
+				(font
+					(size 1.27 1.27)
+				)
+				(hide yes)
+			)
+		)
+		(property "Datasheet" ""
+			(at 242.57 102.87 0)
+			(effects
+				(font
+					(size 1.27 1.27)
+				)
+				(hide yes)
+			)
+		)
+		(property "Description" "Power symbol creates a global label with name \"VDD\""
+			(at 242.57 102.87 0)
+			(effects
+				(font
+					(size 1.27 1.27)
+				)
+				(hide yes)
+			)
+		)
+		(pin "1"
+		)
+		(instances
+			(project ""
+				(path "/cb287dda-24c2-4519-beaf-f97d5ec0b0ad"
+					(reference "#PWR08")
+					(unit 1)
+				)
